File: Science Signals Booster/Science Signals Booster.sch (KiCad schematic (older format))
At the start: 40 parts, among them U1 Molex_SL-2, U10 LB1930MC, U11 Molex_SL-10, U12 Molex_SL_2, U13 Molex_SL_5, U2 Molex_SL-2, U3 5V OKI, U4 OPA320, U5 OPA320, U6 5V OKI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

Commit message: Added a few additional notes in the schematic for clarity
Parts:
- C1, C10, C11, C12, C13, C2: footprint (none) -> Capacitors_SMD:C_0805_HandSoldering
- PWR1: footprint (none) -> LEDs:LED_1206_HandSoldering
- U10: footprint (none) -> MRDT_ICs.pretty:SOIC-10NB
- U8: footprint (none) -> TO_SOT_Packages_SMD:TO-263-6
Other:
- note added: "Need TIVA pins selected for IN1, IN2\n(This implementation is based on last years\nboard which connected to the same motor)"
- note removed: "Need TIVA pins selected for IN1, IN2"
Changed lines of the file:
@@
 F 0 "C1" H 3625 3000 50  0000 L CNN
 F 1 "10uF" H 3625 2800 50  0000 L CNN
-F 2 "" H 3638 2750 50  0001 C CNN
+F 2 "Capacitors_SMD:C_0805_HandSoldering" H 3638 2750 50  0001 C CNN
 F 3 "" H 3600 2900 50  0001 C CNN
 	1    3600 2900
@@
 F 0 "C2" H 3625 3400 50  0000 L CNN
 F 1 "22uF" H 3625 3200 50  0000 L CNN
-F 2 "" H 3638 3150 50  0001 C CNN
+F 2 "Capacitors_SMD:C_0805_HandSoldering" H 3638 3150 50  0001 C CNN
 F 3 "" H 3600 3300 50  0001 C CNN
 	1    3600 3300
@@
 F 0 "PWR1" H 3500 3850 50  0000 C CNN
 F 1 "LED" H 3500 3650 50  0000 C CNN
-F 2 "" H 3500 3750 50  0001 C CNN
+F 2 "LEDs:LED_1206_HandSoldering" H 3500 3750 50  0001 C CNN
 F 3 "" H 3500 3750 50  0001 C CNN
 	1    3500 3750
@@
 F 0 "C10" H 6025 3000 50  0000 L CNN
 F 1 "10uF" H 6025 2800 50  0000 L CNN
-F 2 "" H 6038 2750 50  0001 C CNN
+F 2 "Capacitors_SMD:C_0805_HandSoldering" H 6038 2750 50  0001 C CNN
 F 3 "" H 6000 2900 50  0001 C CNN
 	1    6000 2900
@@
 F 0 "C11" H 6025 3400 50  0000 L CNN
 F 1 "22uF" H 6025 3200 50  0000 L CNN
-F 2 "" H 6038 3150 50  0001 C CNN
+F 2 "Capacitors_SMD:C_0805_HandSoldering" H 6038 3150 50  0001 C CNN
 F 3 "" H 6000 3300 50  0001 C CNN
 	1    6000 3300
@@
 F 0 "U8" H 10150 7800 60  0000 C CNN
 F 1 "BA00DD0WHFP" H 10450 8450 60  0000 C CNN
-F 2 "" H 10450 8050 60  0001 C CNN
+F 2 "TO_SOT_Packages_SMD:TO-263-6" H 10450 8050 60  0001 C CNN
 F 3 "" H 10450 8050 60  0001 C CNN
 	1    10450 8050
@@
 F 0 "C12" H 8875 8500 50  0000 L CNN
 F 1 "33uF" H 8875 8300 50  0000 L CNN
-F 2 "" H 8888 8250 50  0001 C CNN
+F 2 "Capacitors_SMD:C_0805_HandSoldering" H 8888 8250 50  0001 C CNN
 F 3 "" H 8850 8400 50  0001 C CNN
 	1    8850 8400
@@
 F 0 "C13" H 11875 8500 50  0000 L CNN
 F 1 "22uF" H 11875 8300 50  0000 L CNN
-F 2 "" H 11888 8250 50  0001 C CNN
+F 2 "Capacitors_SMD:C_0805_HandSoldering" H 11888 8250 50  0001 C CNN
 F 3 "" H 11850 8400 50  0001 C CNN
 	1    11850 8400
@@
 F 0 "U10" H 12300 2000 49  0000 C CNN
 F 1 "LB1930MC" H 12550 2500 49  0000 C CNN
-F 2 "" H 12500 2200 49  0001 C CNN
+F 2 "MRDT_ICs.pretty:SOIC-10NB" H 12500 2200 49  0001 C CNN
 F 3 "" H 12500 2200 49  0001 C CNN
 	1    12500 2200
@@
 Text Notes 10850 1700 0    98   ~ 0
 Spectrometer Motor
-Text Notes 10900 2650 0    39   ~ 0
-Need TIVA pins selected for IN1, IN2
+Text Notes 10900 2750 0    39   ~ 0
+Need TIVA pins selected for IN1, IN2\n(This implementation is based on last years\nboard which connected to the same motor)
 Wire Wire Line
 	9750 3550 9450 3550

Commit message: Finalised schematic and began working on board layout
Parts:
- removed C1, C10: 10uF, Capacitors_SMD:C_0805_HandSoldering, symbol CP
- removed C11, C13, C2: 22uF, Capacitors_SMD:C_0805_HandSoldering, symbol CP
- removed C12: 33uF, Capacitors_SMD:C_0805_HandSoldering, symbol CP
- removed C14, C3, C4: 1uF, Capacitors_SMD:C_0805_HandSoldering, symbol CP
- removed C5, C6: 2.7pF, Capacitors_SMD:C_0805_HandSoldering, symbol CP
- removed C8, C9: 0.1uF, Capacitors_SMD:C_0805_HandSoldering, symbol CP
- added C1, C10, C11, C2: 10uF, Capacitors_SMD:C_0603_HandSoldering, symbol C
- added C12: 33uF, Capacitors_SMD:C_0603_HandSoldering, symbol C
- added C13: 22uF, Capacitors_SMD:C_0603_HandSoldering, symbol C
- added C14, C3, C4: 1uF, Capacitors_SMD:C_0603_HandSoldering, symbol C
- added C5, C6: 2.7pF, Capacitors_SMD:C_0603_HandSoldering, symbol C
- added C8, C9: .1uF, Capacitors_SMD:C_0603_HandSoldering, symbol C
- C7: footprint MRDT_Connectors.pretty:Anderson_3_Horisontal_Side_by_Side -> MRDT_Connectors:Anderson_3_Horisontal_Side_by_Side
- R1: value 1k -> 500; footprint Resistors_SMD:R_0805_HandSoldering -> Resistors_SMD:R_0603_HandSoldering
- R10, R11, R12, R2, R3, R4, R5, R6, R7, R8, R9: footprint Resistors_SMD:R_0805_HandSoldering -> Resistors_SMD:R_0603_HandSoldering
- U1, U12, U2, U9: footprint MRDT_Connectors.pretty:MOLEX_SL_2 -> MRDT_Connectors:MOLEX_SL_2_Horizontal
- U10: footprint MRDT_ICs.pretty:SOIC-10NB -> Housings_SSOP:TSSOP-20_4.4x6.5mm_Pitch0.65mm
- U11: footprint MRDT_Connectors.pretty:MOLEX_SL_10 -> MRDT_Connectors:MOLEX_SL_10_Horizontal
- U13: footprint MRDT_Connectors.pretty:MOLEX_SL_5 -> MRDT_Connectors:MOLEX_SL_5_Horizontal
- U3, U6: footprint MRDT_Devices.pretty:OKI_Horisontal -> MRDT_Devices:OKI_Horisontal
- U7: footprint MRDT_Shields.pretty:TM4C129E_Launchpad_FULL_Booster -> MRDT_Shields:TM4C129E_Launchpad_FULL_Booster
- U8: footprint TO_SOT_Packages_SMD:TO-263-6 -> TO_SOT_Packages_SMD:TO-252-5_TabPin3
Connections:
- net labels added: LINEAR_ENCODER, Motor_IN1, Motor_IN2, PHOTODIODE_1, PHOTODIODE_2
- net labels removed: LINEAR_ENCODER_T2CCP0, PHOTODIODE_AIN_12, PHOTODIODE_AIN_13
- wire segments 139 -> 137
Other:
- moved on the sheet: U10
