File: Science Signals Booster/Science Signals Booster.sch (KiCad schematic (older format))
At the start: 40 parts, among them U1 Molex_SL-2, U10 LB1930MC, U11 Molex_SL-10, U12 Molex_SL_2, U13 Molex_SL_5, U2 Molex_SL-2, U3 5V OKI, U4 OPA320, U5 OPA320, U6 5V OKI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

Commit message: Finished Board
Connections:
- net +5V is gone; now on net LOGIC-5V: U11.2, U7.+5V (B2_1)
