File: Science Signals Booster/Science Signals Booster.kicad_pcb (KiCad board)
At the start: 2 copper layers, 40 parts, among them U1 Molex_SL-2, U10 LB1930MC, U11 Molex_SL-10, U12 Molex_SL_2, U13 Molex_SL_5, U2 Molex_SL-2, U3 5V OKI, U4 OPA320, U5 OPA320, U6 5V OKI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

Commit message: Finished Board
Parts:
- added G***: LOGO, MRDT_Silkscreens:Andrew_Van_Horn_Sig_15mm, F.Cu at (189.2, 141.0)
- added G***: LOGO, MRDT_Silkscreens:Atlas_Logo_28.6mmX37.3mm, B.Cu at (163.1, 105.7)
- added G***: LOGO, MRDT_Silkscreens:MRDT_Logo_20mm, F.Cu at (163.8, 134.3)
- moved R11 231.7 mm to (234.3, 91.2), turned to 270 degrees
- moved C12 226.1 mm to (237.2, 93.9), turned to 180 degrees
- moved R12 224.0 mm to (237.3, 90.2), turned to 180 degrees
- moved C13 219.1 mm to (237.2, 92.3), turned to 180 degrees
- moved R10 201.6 mm to (237.3, 95.6), turned to 180 degrees
- moved C14 191.5 mm to (203.7, 103.0)
- moved C11 191.3 mm to (203.7, 104.4)
- moved C10 187.5 mm to (199.9, 104.4)
- moved C2 171.5 mm to (192.9, 104.4)
- moved R1 165.0 mm to (183.2, 110.8), turned to 90 degrees
- moved C1 160.5 mm to (189.1, 104.4)
- moved C5 152.0 mm to (162.2, 92.3), turned to 90 degrees
- moved C3 147.7 mm to (161.4, 98.0), turned to 90 degrees
- moved C4 143.7 mm to (151.3, 97.9), turned to 90 degrees
- moved R2 135.4 mm to (157.0, 92.2), turned to 270 degrees
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Connections:
- U11 pad 2: (no net) -> LOGIC-5V
- U7 pad +3V3: Net-(U7-Pad+3V3) -> +3V3
- U7 pad +5V: Net-(U7-Pad+5V) -> LOGIC-5V
Routing:
- net LOGIC-5V: track 0.00 -> 171.2 mm, vias 0 -> 3
- net +3V3: track 0.00 -> 131.5 mm
- net LASER-CTRL_AIN_7: track 0.00 -> 69.8 mm, vias 0 -> 2
- net ACT-12V: track 0.00 -> 52.1 mm
- net PHOTODIODE_1: track 0.00 -> 43.0 mm, vias 0 -> 1
- net PRESSURE_I2C_0-SDA: track 0.00 -> 38.6 mm
- net PRESSURE_I2C_0-SCL: track 0.00 -> 35.0 mm
- net LOGIC-12V: track 0.00 -> 32.7 mm
- net MOTOR_IN1: track 0.00 -> 32.4 mm
- net MOTOR_IN2: track 0.00 -> 29.9 mm
- net TEMP_AIN_4: track 0.00 -> 28.2 mm
- net HUMIDITY_AIN_0: track 0.00 -> 26.3 mm
- net magINCn: track 0.00 -> 25.9 mm
- net LINEAR_ENCODER: track 0.00 -> 25.0 mm
- net magDECn: track 0.00 -> 24.8 mm
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- added copper zone on B.Cu, net GND
Other:
- board outline added: 124.5 x 81.3 mm
- board text added: "Encoder"
- board text added: "Laser"
- board text added: "Motor"
- board text added: "Photo-1"
- board text added: "Photo-2"
- board text added: "Science Board, Rev 1 Mars Rover 2018 Missouri S&T Andrew Van Horn, Shaun McManus"
- board text added: "Sensor Board"
